Commit message: Corrected coordinates

File: urdf/leadsense.xacro (robot description, xacro)
@@ -5,5 +5,5 @@
   <xacro:macro name="sensor_stereocamera" params="parent:='base_link' *origin right_cam_dist:=0.12">
     <link name="leadsense_left_camera">
-      <visual>
+      <!-- <visual>
         <origin xyz="0 0 0" rpy="0 0 0"/>
         <geometry>
@@ -13,9 +13,9 @@
           <color rgba="0.1 0.1 0.1 1"/>
         </material>
-      </visual>
+      </visual> -->
     </link>
     <link name="leadsense_center">
       <visual>
-        <origin xyz="0 0 0" rpy="1.57 0 1.57"/>
+        <origin xyz="0 ${right_cam_dist} 0" rpy="-1.57 0 -1.57"/>
         <geometry>
           <mesh filename="package://leadsense_ros/urdf/leadsenseL.stl" scale="0.001 0.001 0.001"/>
@@ -27,5 +27,5 @@
     </link>
     <link name="leadsense_right_camera">
-      <visual>
+      <!-- <visual>
         <origin xyz="0 0 0" rpy="0 0 0"/>
         <geometry>
@@ -35,5 +35,5 @@
           <color rgba="0.1 0.1 0.1 1"/>
         </material>
-      </visual>
+      </visual> -->
     </link>
     <link name="leadsense_imu_frame">
